Commit message: robot on the table

File: resources/GazeboRosPackages/fh_desc/model.urdf (robot description, URDF)
Before this commit: robot robot, 35 links, 34 joints
Joints:
- joint world_joint: origin xyz=0.0 0 1.1 rpy=0.0 0.0 0 -> xyz=0.0 0 1.002 rpy=0.0 0.0 0

Commit message: load ros param with ros launch, peer's table fix

File: resources/GazeboRosPackages/fh_desc/model.urdf (robot description, URDF)
Before this commit: robot robot, 35 links, 34 joints
Joints:
- joint world_joint: origin xyz=0.0 0 1.002 rpy=0.0 0.0 0 -> xyz=0.0 0 1.032 rpy=0.0 0.0 0
